Commit message: c

File: rover_description/urdf/rover_description.urdf (robot description, URDF)
Before this commit: robot mars_rover, 14 links, 13 joints
Links:
- link wheel1: geometry collision cylinder length=0.144 radius=0.11; visual mesh filename=package://rover_description/meshes/wheel1.STL
- link wheel2: geometry collision cylinder length=0.144 radius=0.11; visual mesh filename=package://rover_description/meshes/wheel2.STL
- link wheel3: geometry collision cylinder length=0.144 radius=0.11; visual mesh filename=package://rover_description/meshes/wheel3.STL
- link wheel4: geometry collision cylinder length=0.144 radius=0.11; visual mesh filename=package://rover_description/meshes/wheel4.STL
Joints:
- joint steer1: limit lower=-1.57 upper=1.57 effort=5 velocity=6.28 -> lower=-1.57 upper=1.57 effort=10 velocity=6.28
- joint steer2: limit lower=-1.57 upper=1.57 effort=5 velocity=6.28 -> lower=-1.57 upper=1.57 effort=10 velocity=6.28
- joint steer4: limit lower=-1.57 upper=1.57 effort=5 velocity=6.28 -> lower=-1.57 upper=1.57 effort=10 velocity=6.28
- joint steer_3: limit lower=-1.57 upper=1.57 effort=5 velocity=6.28 -> lower=-1.57 upper=1.57 effort=10 velocity=6.28

Commit message: blank

File: rover_description/urdf/rover_description.urdf (robot description, URDF)
Before this commit: robot mars_rover, 14 links, 13 joints
Joints:
- joint camera_optical_joint: origin xyz=0.1 0 0.1 rpy=-1.57 0 -1.57 -> xyz=0 0 0 rpy=-1.57 0 -1.57

Commit message: bs

File: rover_description/urdf/rover_description.urdf (robot description, URDF)
Before this commit: robot mars_rover, 14 links, 13 joints
Links:
- added link camera_link_1; collision box size=0.1 0.1 0.1; visual box size=0.1 0.1 0.1
- added link camera_link_2; collision box size=0.1 0.1 0.1; visual box size=0.1 0.1 0.1
- added link camera_optical_link_1
- added link camera_optical_link_2
Joints:
- added joint camera_joint_1: type fixed, parent chassis, child camera_link_1, origin xyz=0 0.24 0.1 rpy=0 0 1.57
- added joint camera_joint_2: type fixed, parent chassis, child camera_link_2, origin xyz=0 -0.24 0.1 rpy=0 0 -1.57
- added joint camera_optical_joint_1: type fixed, parent camera_link_1, child camera_optical_link_1, origin xyz=0 0 0 rpy=-1.57 0 -1.57
- added joint camera_optical_joint_2: type fixed, parent camera_link_2, child camera_optical_link_2, origin xyz=0 0 0 rpy=-1.57 0 -1.57
